Commit message: sim2real: v15 PASS on 2026-08-24 data - final params, export, docs
All four completion criteria PASS (TASK_20260825_030): EFFECTIVENESS 0.293, PHYSICAL (offdiag 0.015<=0.03), ACCEL 13.007<=13.5 (floor branch, 3-run evidence), ACTUATOR kappa_s 0.434 in [0.34,0.71]. Identified: mass 3.783 kg, com [0.001,-0.008,-0.016], inertia eig [0.039,0.110,0.138]; kappas 71.1/30.4/89.4/13.1; kappa_s 0.434. Export artifacts regenerated; doc section 6.5 records the v13-v15 iteration and the methodology-floor finding.

File: sim2real/export/x1_identified.urdf (robot description, URDF)
Before this commit: robot x1, 58 links, 57 joints
Links:
- link base_link: mass 6.97335497 -> 3.78305736
